File: pcb_challenge_final.kicad_pcb (KiCad board)
At the start: 2 copper layers, 154 parts, among them J4 Conn_01x04_Pin, J5 Conn_01x04_Pin, Q12 Q_Dual_NPN_PNP_B1E2B2C2E1C1, Q13 Q_Dual_NPN_PNP_B1E2B2C2E1C1, Q14 Q_Dual_NPN_PNP_B1E2B2C2E1C1, Q15 Q_Dual_NPN_PNP_B1E2B2C2E1C1, Q16 Q_Dual_NPN_PNP_B1E2B2C2E1C1, Q18 Q_Dual_NPN_PNP_B1E2B2C2E1C1, Q19 Q_Dual_NPN_PNP_B1E2B2C2E1C1, Q20 Q_Dual_NPN_PNP_B1E2B2C2E1C1, Q21 Q_Dual_NPN_PNP_B1E2B2C2E1C1, Q22 Q_Dual_NPN_PNP_B1E2B2C2E1C1, Q23 Q_Dual_NPN_PNP_B1E2B2C2E1C1, Q24 Q_Dual_NPN_PNP_B1E2B2C2E1C1, Q25 Q_Dual_NPN_PNP_B1E2B2C2E1C1, Q26 Q_Dual_NPN_PNP_B1E2B2C2E1C1, Q27 Q_Dual_NPN_PNP_B1E2B2C2E1C1, SW2 SW_MEC_5G, U1 74AUP1G80, U10 NMUX1308BQ, U11 NMUX1308BQ, U12 NMUX1308BQ, U13 NMUX1308BQ, U14 NMUX1308BQ, U15 NMUX1308BQ, U16 NMUX1308BQ, U17 74AUP1G80, U18 74AHC1G86, U19 74AUP1G80, U2 NMUX1308BQ, U20 74AUP1G80, U21 74LV1T08GV, U22 CD74HC283M96, U23 74LV1T08GV, U24 74LVC1GU04DRL, U25 ESP32-S3-MINI-1, U26 74LVC1GU04DRL, U27 74LV1T08GV, U28 CD74HC283M96, U29 NMUX1308BQ, U3 74AHC1G86, U30 NMUX1308BQ, U31 NMUX1308BQ, U32 NMUX1308BQ, U33 74AUP1G80, U34 74AUP1G80, U35 NMUX1308BQ, U36 NMUX1308BQ, U37 74AUP1G80, U38 74AUP1G80, U39 NMUX1308BQ, U4 74AUP1G80, U40 NMUX1308BQ, U41 NMUX1308BQ, U42 NMUX1308BQ, U43 NMUX1308BQ, U44 NMUX1308BQ, U45 74AUP1G80, U46 74AUP1G80, U47 74AUP1G80, U48 74AUP1G80, U49 74AUP1G80, U5 74AUP1G80, U50 74AUP1G80, U51 74LV1T08GV, U52 74AHC1G86, U53 74LVC1GU04DRL, U54 74LVC1GU04DRL, U55 74AHC1G86, U56 74AHC1G86, U57 74LVC1GU04DRL, U58 74LVC1GU04DRL, U59 74LV1T08GV, U6 74AUP1G80, U60 74AHC1G86, U61 74LVC1GU04DRL, U62 74LV1T08GV, U63 74LV1T08GV, U64 NMUX1308BQ, U65 74AUP1G80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

Commit message: New updated file
Parts:
- removed Q12, Q13, Q14: Q_Dual_NPN_PNP_B1E2B2C2E1C1, Package_TO_SOT_SMD:SOT-1123
- added C1: 22uF, Capacitor_SMD:C_0201_0603Metric, F.Cu at (191.8, 146.7)
- added C2: 0.1uF, Capacitor_SMD:C_0201_0603Metric, F.Cu at (191.8, 148.5)
- added C3: 12pF, Capacitor_SMD:C_0201_0603Metric, F.Cu at (191.8, 150.2)
- added C4: 12pF, Capacitor_SMD:C_0201_0603Metric, F.Cu at (191.8, 152.0)
- added C5: 22pF, Capacitor_SMD:C_0201_0603Metric, F.Cu at (191.8, 153.7)
- added C6: 22pF, Capacitor_SMD:C_0201_0603Metric, F.Cu at (191.8, 155.5)
- added C7: 22uF, Capacitor_SMD:C_0201_0603Metric, F.Cu at (191.8, 157.2)
- added C8: 0.1uF, Capacitor_SMD:C_0201_0603Metric, F.Cu at (191.8, 159.0)
- added Q17: Q_Dual_NPN_PNP_B1E2B2C2E1C1, Package_TO_SOT_SMD:SOT-1123, F.Cu at (170.1, 100.4)
- added Q28: Q_Dual_NPN_PNP_B1E2B2C2E1C1, Package_TO_SOT_SMD:SOT-1123, F.Cu at (176.1, 102.6)
- added Q29: Q_Dual_NPN_PNP_B1E2B2C2E1C1, Package_TO_SOT_SMD:SOT-1123, F.Cu at (176.1, 104.8)
- added R1: 10k, Capacitor_SMD:C_0402_1005Metric, F.Cu at (197.4, 158.4)
- added SW1: SW_Push, Button_Switch_SMD:SW_DIP_SPSTx01_Slide_6.7x4.1mm_W8.61mm_P2.54mm_LowProfile, F.Cu at (199.3, 148.8)
- added SW3: SW_Push, Button_Switch_SMD:SW_DIP_SPSTx01_Slide_6.7x4.1mm_W8.61mm_P2.54mm_LowProfile, F.Cu at (199.3, 154.5)
- moved D1 185.2 mm to (177.8, 139.2)
- moved U9 180.2 mm to (181.5, 123.4)
- moved U66 171.3 mm to (154.1, 146.5)
- moved Y1 167.6 mm to (133.9, 152.2)
- moved R61 165.8 mm to (137.3, 130.8)
- moved R62 165.8 mm to (137.3, 133.3)
- moved Y2 165.6 mm to (176.9, 111.3)
- moved U67 159.5 mm to (154.1, 149.1)
- moved R64 156.0 mm to (137.3, 138.4)
- moved R63 156.0 mm to (137.3, 135.9)
- moved U24 153.4 mm to (174.8, 144.8)
- moved U57 153.4 mm to (178.3, 144.8)
- moved U58 153.4 mm to (178.3, 148.0)
- moved U61 153.4 mm to (178.3, 151.2)
- moved J4 153.1 mm to (168.0, 111.4)
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Connections:
- Q15 pad 2: (no net) -> b4
- Q15 pad 3: (no net) -> Net-(Q15A-E1)
- Q16 pad 2: (no net) -> Net-(Q16A-C1)
- Q16 pad 3: (no net) -> Net-(Q16A-E1)
- Q18 pad 2: (no net) -> rw3
- Q18 pad 3: (no net) -> Net-(Q18A-E1)
- Q19 pad 2: (no net) -> rw2
- Q19 pad 3: (no net) -> Net-(Q19A-E1)
- Q20 pad 2: (no net) -> rw1
- Q20 pad 3: (no net) -> Net-(Q20A-E1)
- Q21 pad 2: (no net) -> wr3
- Q21 pad 3: (no net) -> Net-(Q21A-E1)
- Q22 pad 2: (no net) -> wr2
- Q22 pad 3: (no net) -> Net-(Q22A-E1)
- Q23 pad 2: (no net) -> wr1
- Q23 pad 3: (no net) -> Net-(Q23A-E1)
- Q24 pad 2: (no net) -> Net-(Q24A-C1)
- Q24 pad 3: (no net) -> Net-(Q24A-E1)
- Q25 pad 2: (no net) -> Net-(Q25A-C1)
- Q25 pad 3: (no net) -> Net-(Q25A-E1)
- Q26 pad 2: (no net) -> Net-(Q26A-C1)
- Q26 pad 3: (no net) -> Net-(Q26A-E1)
- Q27 pad 2: (no net) -> Net-(Q27A-C1)
- Q27 pad 3: (no net) -> Net-(Q27A-E1)
- R36 pad 2: Net-(Q18A-E1) -> Net-(Q20A-E1)
- R40 pad 2: Net-(Q20A-E1) -> Net-(Q18A-E1)
- R7 pad 2: CLK -> clk
- U25 pad 3: 3v3 -> +3.3V
- Y2 pad 3: CLK -> clk

Commit message: Updated the latest version of segregated components on PCB
Parts:
- moved U9 185.8 mm to (25.5, 22.5)
- moved D1 184.0 mm to (26.9, 33.8)
- moved Q29 170.3 mm to (22.9, 179.3)
- moved U66 167.8 mm to (270.7, 25.8)
- moved Y2 167.3 mm to (22.2, 47.4)
- moved R61 164.6 mm to (266.2, 28.5)
- moved R62 164.6 mm to (266.2, 31.0)
- moved Q28 162.9 mm to (32.9, 180.3)
- moved R63 153.8 mm to (261.6, 45.3)
- moved R64 153.8 mm to (261.6, 47.8)
- moved J4 152.0 mm to (22.0, 153.9)
- moved J5 152.0 mm to (26.6, 153.9)
- moved U67 152.0 mm to (269.8, 50.5)
- moved GREEN_LED1 150.5 mm to (85.3, 23.0)
- moved Q17 149.1 mm to (43.9, 179.8)
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